File: kicad/newcricket.sch (KiCad schematic (older format))
At the start: 23 parts, among them IC1 ATTINY85-P, Q1 Q_NPN_BCE, SW1 SW_PUSH, SW2 SW_PUSH, SW3 SWITCH_INV, U1 LM335, U2 78L05

Commit message: added missing ground
Connections:
- net GND: now also RV1.1
Changed lines of the file:
@@
 LIBS:contrib
 LIBS:valves
-LIBS:capteurs
 LIBS:newcricket-cache
 EELAYER 25 0
@@
 $EndComp
 $Comp
-L VCC #PWR06
-U 1 1 565B75C3
-P 3050 2600
-F 0 "#PWR06" H 3050 2450 50  0001 C CNN
-F 1 "VCC" H 3050 2750 50  0000 C CNN
-F 2 "" H 3050 2600 50  0000 C CNN
-F 3 "" H 3050 2600 50  0000 C CNN
-	1    3050 2600
-	1    0    0    -1
-$EndComp
-$Comp
 L VCC #PWR07
 U 1 1 565B75FE
@@
 Wire Wire Line
 	2100 4050 2100 4100
+Wire Wire Line
+	3200 4900 3200 5050
+Wire Wire Line
+	3200 5050 3550 5050
+Connection ~ 3550 5050
+$Comp
+L VCC #PWR06
+U 1 1 565B75C3
+P 3050 2600
+F 0 "#PWR06" H 3050 2450 50  0001 C CNN
+F 1 "VCC" H 3050 2750 50  0000 C CNN
+F 2 "" H 3050 2600 50  0000 C CNN
+F 3 "" H 3050 2600 50  0000 C CNN
+	1    3050 2600
+	1    0    0    -1
+$EndComp
 $EndSCHEMATC
